File: pcb/tiny-keeb/tiny-keeb.kicad_sch (KiCad schematic)
At the start: 123 parts, among them J2 Conn_01x20_Socket, SW1 SW_RCTRL, SW10 SW_A, SW11 SW_X, SW12 SW_LWIN, SW13 SW_2, SW14 SW_E, SW15 SW_S, SW16 SW_C, SW17 SW_LALT, SW18 SW_', SW19 SW_3, SW2 SW_ESC, SW20 SW_R, SW21 SW_D, SW22 SW_V, SW23 SW_Z, SW24 SW_/, SW25 SW_4, SW26 SW_T, SW27 SW_F, SW28 SW_B, SW29 SW_-, SW3 SW_TAB, SW31 SW_5, SW32 SW_Y, SW33 SW_G, SW34 SW_N, SW35 SW_], SW37 SW_6, SW38 SW_U, SW39 SW_H, SW4 SW_CAPS, SW40 SW_M, SW41 SW_SPACE, SW43 SW_7, SW44 SW_I, SW45 SW_J, SW46 SW_,, SW49 SW_8, SW5 SW_LSHIFT, SW50 SW_O, SW51 SW_K, SW52 SW_., SW55 SW_9, SW56 SW_P, SW57 SW_L, SW58 SW_RSHIFT, SW59 SW_RALT, SW6 SW_LCTRL, SW61 SW_0, SW62 SW_[, SW63 SW_;, SW65 SW_RWIN, SW66 SW_FN, SW67 SW_=, SW7 SW_Q, SW72 SW_BACKSPACE, SW73 SW_\, SW74 SW_ENTER, SW8 SW_1, SW9 SW_W

Commit message: pcb close to done, housing in progress, caps not started
Connections:
- net GND: now also J2.1 (Pin_1); no longer J2.20 (Pin_20)
- net col0: now also J2.15 (Pin_15); no longer J2.6 (Pin_6)
- net col1: now also J2.14 (Pin_14); no longer J2.7 (Pin_7)
- net col10: now also J2.5 (Pin_5); no longer J2.16 (Pin_16)
- net col11: now also J2.4 (Pin_4); no longer J2.17 (Pin_17)
- net col12: now also J2.3 (Pin_3); no longer J2.18 (Pin_18)
- net col13: now also J2.2 (Pin_2); no longer J2.19 (Pin_19)
- net col2: now also J2.13 (Pin_13); no longer J2.8 (Pin_8)
- net col3: now also J2.12 (Pin_12); no longer J2.9 (Pin_9)
- net col4: now also J2.11 (Pin_11); no longer J2.10 (Pin_10)
- net col5: now also J2.10 (Pin_10); no longer J2.11 (Pin_11)
- net col6: now also J2.9 (Pin_9); no longer J2.12 (Pin_12)
- net col7: now also J2.8 (Pin_8); no longer J2.13 (Pin_13)
- net col8: now also J2.7 (Pin_7); no longer J2.14 (Pin_14)
- net col9: now also J2.6 (Pin_6); no longer J2.15 (Pin_15)
- net row0: now also J2.20 (Pin_20); no longer J2.1 (Pin_1)
- net row1: now also J2.19 (Pin_19); no longer J2.2 (Pin_2)
- net row2: now also J2.18 (Pin_18); no longer J2.3 (Pin_3)
- net row3: now also J2.17 (Pin_17); no longer J2.4 (Pin_4)
- net row4: now also J2.16 (Pin_16); no longer J2.5 (Pin_5)
Changed lines of the file:
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@@
     )
   )
-  (symbol (lib_id "Connector:Conn_01x20_Socket") (at 53.34 135.89 0) (unit 1)
-    (in_bom yes) (on_board yes) (dnp no) (fields_autoplaced)
-    (property "Reference" "J2" (at 54.61 135.89 0)
+  (symbol (lib_id "Connector:Conn_01x20_Socket") (at 53.34 138.43 0) (mirror x) (unit 1)
+    (in_bom yes) (on_board yes) (dnp no)
+    (property "Reference" "J2" (at 54.61 138.43 0)
       (effects (font (size 1.27 1.27)) (justify left))
     )
-    (property "Value" "Conn_01x20_Socket" (at 54.61 138.43 0)
+    (property "Value" "Conn_01x20_Socket" (at 54.61 135.89 0)
       (effects (font (size 1.27 1.27)) (justify left))
     )
-    (property "Footprint" "Connector_PinSocket_2.54mm:PinSocket_1x20_P2.54mm_Vertical" (at 53.34 135.89 0)
+    (property "Footprint" "Connector_PinSocket_2.54mm:PinSocket_1x20_P2.54mm_Vertical" (at 53.34 138.43 0)
       (effects (font (size 1.27 1.27)) hide)
     )
-    (property "Datasheet" "~" (at 53.34 135.89 0)
+    (property "Datasheet" "~" (at 53.34 138.43 0)
       (effects (font (size 1.27 1.27)) hide)
     )

Commit message: finished housing, keycaps, and pcb - waiting to order switches and pcb
Parts:
- added SW30: SW_SPACE2, Button_Switch_THT:SW_PUSH_6mm_square_top, symbol Switch:SW_Push
- SW1, SW10, SW11, SW12, SW13, SW14, SW15, SW16, SW17, SW18, SW19, SW2, SW20, SW21, SW22, SW23, SW24, SW25, SW26, SW27, SW28, SW29, SW3, SW31, SW32, SW33, SW34, SW35, SW37, SW38, SW39, SW4, SW40, SW41, SW43, SW44, SW45, SW46, SW49, SW5, SW50, SW51, SW52, SW55, SW56, SW57, SW58, SW59, SW6, SW61, SW62, SW63, SW65, SW66, SW67, SW7, SW72, SW73, SW74, SW8, SW9: footprint Button_Switch_THT:SW_PUSH_6mm -> Button_Switch_THT:SW_PUSH_6mm_square_top
Connections:
- net col6: now also SW30.1
- net at D41.2 (A), SW41.1: now also SW30.2
